File: PCB/acquisition.sch (KiCad schematic (older format))
At the start: 16 parts, among them J1 Conn_01x02, J2 Accelerometer, U1 RC1602A, U2 MCP601-xP, U3 Arduino_Nano_v3.x, U4 MCP601-xP

Commit message: Ajout du PCB Mise à jour du code arduino et du code python
Parts:
- removed U1: RC1602A, Display:RC1602A, symbol Display_Character:RC1602A
- added J1: Coil, Connector_PinHeader_2.54mm:PinHeader_1x02_P2.54mm_Vertical, symbol Connector_Generic:Conn_01x02
- added J4: LCD, Connector_PinHeader_2.54mm:PinHeader_1x10_P2.54mm_Vertical, symbol Connector_Generic:Conn_01x10
- added RV1: 10k, Potentiometer_THT:Potentiometer_Bourns_3296W_Vertical, symbol Device:R_POT
- C1: footprint (none) -> Capacitor_THT:CP_Radial_D10.0mm_P5.00mm
- J2: renamed from J1; value Conn_01x02 -> potentiometer; footprint (none) -> Connector_PinHeader_2.54mm:PinHeader_1x02_P2.54mm_Vertical
- J3: renamed from J2; footprint (none) -> Connector_PinSocket_2.54mm:PinSocket_1x05_P2.54mm_Vertical
- R1, R2, R3, R4, R5, R6, R7: footprint (none) -> Resistor_THT:R_Axial_DIN0207_L6.3mm_D2.5mm_P10.16mm_Horizontal
- R8: value 2k -> 51k; footprint (none) -> Resistor_THT:R_Axial_DIN0207_L6.3mm_D2.5mm_P10.16mm_Horizontal
- R9: value 51k -> 2k; footprint (none) -> Resistor_THT:R_Axial_DIN0207_L6.3mm_D2.5mm_P10.16mm_Horizontal
- U1: renamed from U2; value MCP601-xP -> MCP6271
- U2: renamed from U4; value MCP601-xP -> MCP6271
Connections:
- net labels added: DB4, DB5, DB6, DB7, Enable, R-W, RS, VDD, VO
- wire segments 51 -> 60
- no-connect marks 2 -> 16
Other:
- moved on the sheet: J2
